Commit message: fix: 新增小车模型仿真全向轮

File: urdf/sim_robot.urdf.xacro (robot description, xacro)
@@ -33,5 +33,5 @@
     <origin xyz="0 0 0.17" rpy="0 0 0"/>
   </joint>
-  <link name="left_wheel_link">
+  <link name="front_left_wheel_link">
     <inertial>
       <mass value="0.6"/>
@@ -55,11 +55,16 @@
     </collision>
   </link>
-  <joint name="left_wheel_joint" type="continuous">
-    <parent link="base_link"/>
-    <child link="left_wheel_link"/>
-    <origin xyz="0 0.19 -0.07" rpy="0 0 0"/>
+  <joint name="front_left_wheel_joint" type="continuous">
+    <parent link="base_link"/>
+    <child link="front_left_wheel_link"/>
+    <origin xyz="0.17 0.19 -0.07" rpy="0 0 0"/>
     <axis xyz="0 1 0"/>
   </joint>
-  <link name="right_wheel_link">
+  <gazebo reference="front_left_wheel_link">
+    <mu1>0.02</mu1>
+    <mu2>1.0</mu2>
+    <fdir1>0.7071068 0 -0.7071068</fdir1>
+  </gazebo>
+  <link name="rear_right_wheel_link">
     <inertial>
       <mass value="0.6"/>
@@ -83,60 +88,81 @@
     </collision>
   </link>
-  <joint name="right_wheel_joint" type="continuous">
-    <parent link="base_link"/>
-    <child link="right_wheel_link"/>
-    <origin xyz="0 -0.19 -0.07" rpy="0 0 0"/>
+  <joint name="rear_right_wheel_joint" type="continuous">
+    <parent link="base_link"/>
+    <child link="rear_right_wheel_link"/>
+    <origin xyz="-0.17 -0.19 -0.07" rpy="0 0 0"/>
     <axis xyz="0 1 0"/>
   </joint>
-  <link name="front_caster_link">
-    <inertial>
-      <mass value="0.1"/>
-      <origin xyz="0 0 0"/>
-      <inertia ixx="0.000064" ixy="0" ixz="0" iyy="0.000064" iyz="0" izz="0.000064"/>
-    </inertial>
-    <visual>
-      <geometry>
-        <sphere radius="0.04"/>
-      </geometry>
-      <material name="caster_gray">
-        <color rgba="0.35 0.35 0.35 1"/>
-      </material>
-    </visual>
-    <collision>
-      <geometry>
-        <sphere radius="0.04"/>
-      </geometry>
-    </collision>
-  </link>
-  <joint name="front_caster_joint" type="fixed">
-    <parent link="base_link"/>
-    <child link="front_caster_link"/>
-    <origin xyz="0.17 0 -0.13" rpy="0 0 0"/>
-  </joint>
-  <link name="rear_caster_link">
-    <inertial>
-      <mass value="0.1"/>
-      <origin xyz="0 0 0"/>
-      <inertia ixx="0.000064" ixy="0" ixz="0" iyy="0.000064" iyz="0" izz="0.000064"/>
-    </inertial>
-    <visual>
-      <geometry>
-        <sphere radius="0.04"/>
-      </geometry>
-      <material name="caster_gray">
-        <color rgba="0.35 0.35 0.35 1"/>
-      </material>
-    </visual>
-    <collision>
-      <geometry>
-        <sphere radius="0.04"/>
-      </geometry>
-    </collision>
-  </link>
-  <joint name="rear_caster_joint" type="fixed">
-    <parent link="base_link"/>
-    <child link="rear_caster_link"/>
-    <origin xyz="-0.17 0 -0.13" rpy="0 0 0"/>
-  </joint>
+  <gazebo reference="rear_right_wheel_link">
+    <mu1>0.02</mu1>
+    <mu2>1.0</mu2>
+    <fdir1>0.7071068 0 -0.7071068</fdir1>
+  </gazebo>
+  <link name="front_right_wheel_link">
+    <inertial>
+      <mass value="0.6"/>
+      <origin xyz="0 0 0"/>
+      <inertia ixx="0.0036" ixy="0" ixz="0" iyy="0.003" iyz="0" izz="0.0036"/>
+    </inertial>
+    <visual>
+      <origin xyz="0 0 0" rpy="1.5707963 0 0"/>
+      <geometry>
+        <cylinder radius="0.10" length="0.05"/>
+      </geometry>
+      <material name="wheel_black">
+        <color rgba="0.08 0.08 0.08 1"/>
+      </material>
+    </visual>
+    <collision>
+      <origin xyz="0 0 0" rpy="1.5707963 0 0"/>
+      <geometry>
+        <cylinder radius="0.10" length="0.05"/>
+      </geometry>
+    </collision>
+  </link>
+  <joint name="front_right_wheel_joint" type="continuous">
+    <parent link="base_link"/>
+    <child link="front_right_wheel_link"/>
+    <origin xyz="0.17 -0.19 -0.07" rpy="0 0 0"/>
+    <axis xyz="0 1 0"/>
+  </joint>
+  <gazebo reference="front_right_wheel_link">
+    <mu1>0.02</mu1>
+    <mu2>1.0</mu2>
+    <fdir1>0.7071068 0 0.7071068</fdir1>
+  </gazebo>
+  <link name="rear_left_wheel_link">
+    <inertial>
+      <mass value="0.6"/>
+      <origin xyz="0 0 0"/>
+      <inertia ixx="0.0036" ixy="0" ixz="0" iyy="0.003" iyz="0" izz="0.0036"/>
+    </inertial>
+    <visual>
+      <origin xyz="0 0 0" rpy="1.5707963 0 0"/>
+      <geometry>
+        <cylinder radius="0.10" length="0.05"/>
+      </geometry>
+      <material name="wheel_black">
+        <color rgba="0.08 0.08 0.08 1"/>
+      </material>
+    </visual>
+    <collision>
+      <origin xyz="0 0 0" rpy="1.5707963 0 0"/>
+      <geometry>
+        <cylinder radius="0.10" length="0.05"/>
+      </geometry>
+    </collision>
+  </link>
+  <joint name="rear_left_wheel_joint" type="continuous">
+    <parent link="base_link"/>
+    <child link="rear_left_wheel_link"/>
+    <origin xyz="-0.17 0.19 -0.07" rpy="0 0 0"/>
+    <axis xyz="0 1 0"/>
+  </joint>
+  <gazebo reference="rear_left_wheel_link">
+    <mu1>0.02</mu1>
+    <mu2>1.0</mu2>
+    <fdir1>0.7071068 0 0.7071068</fdir1>
+  </gazebo>
   <link name="imu_link">
     <inertial>
@@ -283,17 +309,13 @@
   </gazebo>
   <gazebo>
-    <plugin filename="gz-sim-diff-drive-system" name="gz::sim::systems::DiffDrive">
-      <left_joint>left_wheel_joint</left_joint>
-      <right_joint>right_wheel_joint</right_joint>
+    <plugin filename="gz-sim-mecanum-drive-system"
+            name="gz::sim::systems::MecanumDrive">
+      <front_left_joint>front_left_wheel_joint</front_left_joint>
+      <front_right_joint>front_right_wheel_joint</front_right_joint>
+      <back_left_joint>rear_left_wheel_joint</back_left_joint>
+      <back_right_joint>rear_right_wheel_joint</back_right_joint>
+      <wheelbase>0.34</wheelbase>
       <wheel_separation>0.38</wheel_separation>
       <wheel_radius>0.10</wheel_radius>
-      <max_linear_acceleration>1.0</max_linear_acceleration>
-      <min_linear_acceleration>-1.0</min_linear_acceleration>
-      <max_angular_acceleration>2.0</max_angular_acceleration>
-      <min_angular_acceleration>-2.0</min_angular_acceleration>
-      <max_linear_velocity>0.8</max_linear_velocity>
-      <min_linear_velocity>-0.8</min_linear_velocity>
-      <max_angular_velocity>2.0</max_angular_velocity>
-      <min_angular_velocity>-2.0</min_angular_velocity>
       <topic>/cmd_vel</topic>
       <odom_topic>/wheel/odometry</odom_topic>

Commit message: feat: 适配gazebo仿真和nav2导航

File: urdf/sim_robot.urdf.xacro (robot description, xacro)
@@ -1,4 +1,5 @@
 <?xml version="1.0"?>
-<robot name="sim_robot_slam" xmlns:xacro="http://www.ros.org/wiki/xacro">
+<robot name="sim_robot_slam" xmlns:xacro="http://www.ros.org/wiki/xacro"
+       xmlns:gz="https://gazebosim.org">
   <link name="base_footprint">
     <inertial>
@@ -62,7 +63,16 @@
   </joint>
   <gazebo reference="front_left_wheel_link">
-    <mu1>0.02</mu1>
-    <mu2>1.0</mu2>
-    <fdir1>0.7071068 0 -0.7071068</fdir1>
+    <!-- Keep roller friction in the chassis frame as the wheel spins. -->
+    <collision>
+      <surface>
+        <friction>
+          <ode>
+            <mu>1.0</mu>
+            <mu2>0.0</mu2>
+            <fdir1 gz:expressed_in="base_footprint">1 -1 0</fdir1>
+          </ode>
+        </friction>
+      </surface>
+    </collision>
   </gazebo>
   <link name="rear_right_wheel_link">
@@ -95,7 +105,15 @@
   </joint>
   <gazebo reference="rear_right_wheel_link">
-    <mu1>0.02</mu1>
-    <mu2>1.0</mu2>
-    <fdir1>0.7071068 0 -0.7071068</fdir1>
+    <collision>
+      <surface>
+        <friction>
+          <ode>
+            <mu>1.0</mu>
+            <mu2>0.0</mu2>
+            <fdir1 gz:expressed_in="base_footprint">1 -1 0</fdir1>
+          </ode>
+        </friction>
+      </surface>
+    </collision>
   </gazebo>
   <link name="front_right_wheel_link">
@@ -128,7 +146,15 @@
   </joint>
   <gazebo reference="front_right_wheel_link">
-    <mu1>0.02</mu1>
-    <mu2>1.0</mu2>
-    <fdir1>0.7071068 0 0.7071068</fdir1>
+    <collision>
+      <surface>
+        <friction>
+          <ode>
+            <mu>1.0</mu>
+            <mu2>0.0</mu2>
+            <fdir1 gz:expressed_in="base_footprint">1 1 0</fdir1>
+          </ode>
+        </friction>
+      </surface>
+    </collision>
   </gazebo>
   <link name="rear_left_wheel_link">
@@ -161,7 +187,15 @@
   </joint>
   <gazebo reference="rear_left_wheel_link">
-    <mu1>0.02</mu1>
-    <mu2>1.0</mu2>
-    <fdir1>0.7071068 0 0.7071068</fdir1>
+    <collision>
+      <surface>
+        <friction>
+          <ode>
+            <mu>1.0</mu>
+            <mu2>0.0</mu2>
+            <fdir1 gz:expressed_in="base_footprint">1 1 0</fdir1>
+          </ode>
+        </friction>
+      </surface>
+    </collision>
   </gazebo>
   <link name="imu_link">

Commit message: fix: 适配样机尺寸的模型和传感器位置

File: urdf/sim_robot.urdf.xacro (robot description, xacro)
@@ -2,4 +2,11 @@
 <robot name="sim_robot_slam" xmlns:xacro="http://www.ros.org/wiki/xacro"
        xmlns:gz="https://gazebosim.org">
+  <!-- Wheel dimensions and sensor origins follow the measured robot geometry.
+       The outer shell and masses remain a simplified approximation. -->
+  <xacro:property name="wheel_radius" value="0.125"/>
+  <xacro:property name="wheel_width" value="0.05"/>
+  <xacro:property name="wheelbase" value="0.580"/>
+  <xacro:property name="wheel_separation" value="0.454"/>
+  <xacro:property name="base_link_height" value="0.2125"/>
   <link name="base_footprint">
     <inertial>
@@ -13,9 +20,9 @@
       <mass value="8.0"/>
       <origin xyz="0 0 0"/>
-      <inertia ixx="0.0833" ixy="0" ixz="0" iyy="0.1733" iyz="0" izz="0.2267"/>
-    </inertial>
-    <visual>
-      <geometry>
-        <box size="0.48 0.32 0.12"/>
+      <inertia ixx="0.121666667" ixy="0" ixz="0" iyy="0.255" iyz="0" izz="0.346666667"/>
+    </inertial>
+    <visual>
+      <geometry>
+        <box size="0.60 0.40 0.15"/>
       </geometry>
       <material name="chassis_blue">
@@ -25,5 +32,5 @@
     <collision>
       <geometry>
-        <box size="0.48 0.32 0.12"/>
+        <box size="0.60 0.40 0.15"/>
       </geometry>
     </collision>
@@ -32,5 +39,5 @@
     <parent link="base_footprint"/>
     <child link="base_link"/>
-    <origin xyz="0 0 0.17" rpy="0 0 0"/>
+    <origin xyz="0 0 ${base_link_height}" rpy="0 0 0"/>
   </joint>
   <link name="front_left_wheel_link">
@@ -38,10 +45,10 @@
       <mass value="0.6"/>
       <origin xyz="0 0 0"/>
-      <inertia ixx="0.0036" ixy="0" ixz="0" iyy="0.003" iyz="0" izz="0.0036"/>
-    </inertial>
-    <visual>
-      <origin xyz="0 0 0" rpy="1.5707963 0 0"/>
-      <geometry>
-        <cylinder radius="0.10" length="0.05"/>
+      <inertia ixx="0.00246875" ixy="0" ixz="0" iyy="0.0046875" iyz="0" izz="0.00246875"/>
+    </inertial>
+    <visual>
+      <origin xyz="0 0 0" rpy="1.5707963 0 0"/>
+      <geometry>
+        <cylinder radius="${wheel_radius}" length="${wheel_width}"/>
       </geometry>
       <material name="wheel_black">
@@ -52,5 +59,5 @@
       <origin xyz="0 0 0" rpy="1.5707963 0 0"/>
       <geometry>
-        <cylinder radius="0.10" length="0.05"/>
+        <cylinder radius="${wheel_radius}" length="${wheel_width}"/>
       </geometry>
     </collision>
@@ -59,5 +66,5 @@
     <parent link="base_link"/>
     <child link="front_left_wheel_link"/>
-    <origin xyz="0.17 0.19 -0.07" rpy="0 0 0"/>
+    <origin xyz="${wheelbase / 2} ${wheel_separation / 2} ${wheel_radius - base_link_height}" rpy="0 0 0"/>
     <axis xyz="0 1 0"/>
   </joint>
@@ -80,10 +87,10 @@
       <mass value="0.6"/>
       <origin xyz="0 0 0"/>
-      <inertia ixx="0.0036" ixy="0" ixz="0" iyy="0.003" iyz="0" izz="0.0036"/>
-    </inertial>
-    <visual>
-      <origin xyz="0 0 0" rpy="1.5707963 0 0"/>
-      <geometry>
-        <cylinder radius="0.10" length="0.05"/>
+      <inertia ixx="0.00246875" ixy="0" ixz="0" iyy="0.0046875" iyz="0" izz="0.00246875"/>
+    </inertial>
+    <visual>
+      <origin xyz="0 0 0" rpy="1.5707963 0 0"/>
+      <geometry>
+        <cylinder radius="${wheel_radius}" length="${wheel_width}"/>
       </geometry>
       <material name="wheel_black">
@@ -94,5 +101,5 @@
       <origin xyz="0 0 0" rpy="1.5707963 0 0"/>
       <geometry>
-        <cylinder radius="0.10" length="0.05"/>
+        <cylinder radius="${wheel_radius}" length="${wheel_width}"/>
       </geometry>
     </collision>
@@ -101,5 +108,5 @@
     <parent link="base_link"/>
     <child link="rear_right_wheel_link"/>
-    <origin xyz="-0.17 -0.19 -0.07" rpy="0 0 0"/>
+    <origin xyz="${-wheelbase / 2} ${-wheel_separation / 2} ${wheel_radius - base_link_height}" rpy="0 0 0"/>
     <axis xyz="0 1 0"/>
   </joint>
@@ -121,10 +128,10 @@
       <mass value="0.6"/>
       <origin xyz="0 0 0"/>
-      <inertia ixx="0.0036" ixy="0" ixz="0" iyy="0.003" iyz="0" izz="0.0036"/>
-    </inertial>
-    <visual>
-      <origin xyz="0 0 0" rpy="1.5707963 0 0"/>
-      <geometry>
-        <cylinder radius="0.10" length="0.05"/>
+      <inertia ixx="0.00246875" ixy="0" ixz="0" iyy="0.0046875" iyz="0" izz="0.00246875"/>
+    </inertial>
+    <visual>
+      <origin xyz="0 0 0" rpy="1.5707963 0 0"/>
+      <geometry>
+        <cylinder radius="${wheel_radius}" length="${wheel_width}"/>
       </geometry>
       <material name="wheel_black">
@@ -135,5 +142,5 @@
       <origin xyz="0 0 0" rpy="1.5707963 0 0"/>
       <geometry>
-        <cylinder radius="0.10" length="0.05"/>
+        <cylinder radius="${wheel_radius}" length="${wheel_width}"/>
       </geometry>
     </collision>
@@ -142,5 +149,5 @@
     <parent link="base_link"/>
     <child link="front_right_wheel_link"/>
-    <origin xyz="0.17 -0.19 -0.07" rpy="0 0 0"/>
+    <origin xyz="${wheelbase / 2} ${-wheel_separation / 2} ${wheel_radius - base_link_height}" rpy="0 0 0"/>
     <axis xyz="0 1 0"/>
   </joint>
@@ -162,10 +169,10 @@
       <mass value="0.6"/>
       <origin xyz="0 0 0"/>
-      <inertia ixx="0.0036" ixy="0" ixz="0" iyy="0.003" iyz="0" izz="0.0036"/>
-    </inertial>
-    <visual>
-      <origin xyz="0 0 0" rpy="1.5707963 0 0"/>
-      <geometry>
-        <cylinder radius="0.10" length="0.05"/>
+      <inertia ixx="0.00246875" ixy="0" ixz="0" iyy="0.0046875" iyz="0" izz="0.00246875"/>
+    </inertial>
+    <visual>
+      <origin xyz="0 0 0" rpy="1.5707963 0 0"/>
+      <geometry>
+        <cylinder radius="${wheel_radius}" length="${wheel_width}"/>
       </geometry>
       <material name="wheel_black">
@@ -176,5 +183,5 @@
       <origin xyz="0 0 0" rpy="1.5707963 0 0"/>
       <geometry>
-        <cylinder radius="0.10" length="0.05"/>
+        <cylinder radius="${wheel_radius}" length="${wheel_width}"/>
       </geometry>
     </collision>
@@ -183,5 +190,5 @@
     <parent link="base_link"/>
     <child link="rear_left_wheel_link"/>
-    <origin xyz="-0.17 0.19 -0.07" rpy="0 0 0"/>
+    <origin xyz="${-wheelbase / 2} ${wheel_separation / 2} ${wheel_radius - base_link_height}" rpy="0 0 0"/>
     <axis xyz="0 1 0"/>
   </joint>
@@ -217,13 +224,15 @@
     <parent link="base_link"/>
     <child link="imu_link"/>
-    <origin xyz="0 0 0.02" rpy="0 0 0"/>
+    <origin xyz="-0.1955 0 ${0.368 - base_link_height}" rpy="0 0 0"/>
   </joint>
   <link name="lidar_link">
     <inertial>
       <mass value="0.35"/>
-      <origin xyz="0 0 0"/>
+      <origin xyz="0 0 0.035"/>
       <inertia ixx="0.0006" ixy="0" ixz="0" iyy="0.0006" iyz="0" izz="0.001"/>
     </inertial>
     <visual>
+      <!-- The supplied 0.539 m height is the LiDAR mounting-frame height. -->
+      <origin xyz="0 0 0.035"/>
       <geometry>
         <cylinder radius="0.055" length="0.07"/>
@@ -237,5 +246,5 @@
     <parent link="base_link"/>
     <child link="lidar_link"/>
-    <origin xyz="0 0 0.13" rpy="0 0 0"/>
+    <origin xyz="0.343 0 ${0.539 - base_link_height}" rpy="0 0 0"/>
   </joint>
   <gazebo reference="imu_link">
@@ -349,7 +358,7 @@
       <back_left_joint>rear_left_wheel_joint</back_left_joint>
       <back_right_joint>rear_right_wheel_joint</back_right_joint>
-      <wheelbase>0.34</wheelbase>
-      <wheel_separation>0.38</wheel_separation>
-      <wheel_radius>0.10</wheel_radius>
+      <wheelbase>${wheelbase}</wheelbase>
+      <wheel_separation>${wheel_separation}</wheel_separation>
+      <wheel_radius>${wheel_radius}</wheel_radius>
       <topic>/cmd_vel</topic>
       <odom_topic>/wheel/odometry</odom_topic>
